File: Maple_Mini_Template.sch (KiCad schematic (older format))
At the start: 1 part

Commit message: assign footprints
Parts:
- removed P?: CONN_01X06, symbol CONN_01X06
Changed lines of the file:
@@
 F5 "5V" I L 7875 1725 60
 $EndSheet
-$Comp
-L CONN_01X06 P?
-U 1 1 57F7E8D7
-P 5150 3625
-F 0 "P?" H 5150 3975 50  0000 C CNN
-F 1 "CONN_01X06" V 5250 3625 50  0000 C CNN
-F 2 "" H 5150 3625 60  0000 C CNN
-F 3 "" H 5150 3625 60  0000 C CNN
-	1    5150 3625
-	1    0    0    -1
-$EndComp
 $EndSCHEMATC

Commit message: bug fix
Parts:
- added P?: CONN_01X06, symbol CONN_01X06
Changed lines of the file:
@@
 F5 "5V" I L 7875 1725 60
 $EndSheet
+$Comp
+L CONN_01X06 P?
+U 1 1 57F7E8D7
+P 5150 3625
+F 0 "P?" H 5150 3975 50  0000 C CNN
+F 1 "CONN_01X06" V 5250 3625 50  0000 C CNN
+F 2 "" H 5150 3625 60  0000 C CNN
+F 3 "" H 5150 3625 60  0000 C CNN
+	1    5150 3625
+	1    0    0    -1
+$EndComp
 $EndSCHEMATC
