File: Maple_mini.sch (KiCad schematic (older format))
At the start: 24 parts, among them P1 CONN_01X03, Q1 Q_NPN_BEC, Q2 Q_NPN_BEC, SW1 SW_PUSH, SW2 SW_PUSH, U1 STM32F103CBT6, X1 CRYSTAL_SMD

Commit message: assign footprints
Parts:
- C1, C2: footprint (none) -> Capacitors_SMD:C_0603
- C3, C4, C5, C6: value C -> 1uF; footprint (none) -> Capacitors_SMD:C_0603
- D1: footprint (none) -> LEDs:LED_0805
- P1: footprint (none) -> Socket_Strips:Socket_Strip_Straight_1x03
- Q1, Q2: footprint (none) -> TO_SOT_Packages_SMD:SOT-23
- R1: footprint (none) -> Resistors_SMD:R_0603_HandSoldering; Part # 311-1.0KARCT-ND -> 311-1.0KGRCT-ND
- R10, R9: footprint (none) -> Resistors_SMD:R_0603_HandSoldering; Part # RMCF0805JT22R0CT-ND -> 311-22GRCT-ND
- R2: footprint (none) -> Resistors_SMD:R_0603_HandSoldering; Part # 311-330ARCT-ND -> 311-330GRCT-ND
- R3: footprint (none) -> Resistors_SMD:R_0603_HandSoldering; Part # RMCF0805JT47K0CT-ND -> 311-47KGRCT-ND
- R4, R6, R7: footprint (none) -> Resistors_SMD:R_0603_HandSoldering; Part # RMCF0805JT10K0CT-ND -> 311-10KGRCT-ND
- R5: footprint (none) -> Resistors_SMD:R_0603_HandSoldering; Part # RMCF0805JT36K0CT-ND -> 311-36KGRCT-ND
- R8: footprint (none) -> Resistors_SMD:R_0603_HandSoldering; Part # RMCF0805JT1K50CT-ND -> 311-1.5KGRCT-ND
- SW1, SW2: footprint (none) -> KiCad_Footprint:smd_push
- U1: footprint LQFP48 -> Housings_QFP:LQFP-48_7x7mm_Pitch0.5mm
- X1: footprint (none) -> KiCad_Footprint:crystal_maple
