File: Maple_mini.sch (KiCad schematic (older format))
At the start: 24 parts, among them P1 CONN_01X03, Q1 Q_NPN_BEC, Q2 Q_NPN_BEC, SW1 SW_PUSH, SW2 SW_PUSH, U1 STM32F103CBT6, X1 CRYSTAL_SMD

Commit message: test
Parts:
- C1, C2: value C -> 18pF
Changed lines of the file:
@@
 P 900 2850
 F 0 "C1" H 925 2950 50  0000 L CNN
-F 1 "C" H 925 2750 50  0000 L CNN
+F 1 "18pF" H 925 2750 50  0000 L CNN
 F 2 "" H 938 2700 50  0000 C CNN
 F 3 "" H 900 2850 50  0000 C CNN
@@
 P 900 3250
 F 0 "C2" H 925 3350 50  0000 L CNN
-F 1 "C" H 925 3150 50  0000 L CNN
+F 1 "18pF" H 925 3150 50  0000 L CNN
 F 2 "" H 938 3100 50  0000 C CNN
 F 3 "" H 900 3250 50  0000 C CNN
